Commit message: added pidf setup to non flying urdf as well

File: laika_ws/src/laika_sim/urdf/laika.xacro.urdf (robot description, URDF)
Before this commit: robot laika, 14 links, 13 joints
Links:
- added link bl_sphere; collision sphere radius=0.02; visual sphere radius=0.02
- added link br_sphere; collision sphere radius=0.02; visual sphere radius=0.02
- added link fl_sphere; collision sphere radius=0.02; visual sphere radius=0.02
- added link fr_sphere; collision sphere radius=0.02; visual sphere radius=0.02
Joints:
- added joint bl_foot: type fixed, parent bl_lower_link, child bl_sphere, origin xyz=-0.4 -0.05 0.015 rpy=0 0 0
- added joint br_foot: type fixed, parent br_lower_link, child br_sphere, origin xyz=-0.4 -0.05 0.015 rpy=0 0 0
- added joint fl_foot: type fixed, parent fl_lower_link, child fl_sphere, origin xyz=-0.4 -0.05 0.015 rpy=0 0 0
- added joint fr_foot: type fixed, parent fr_lower_link, child fr_sphere, origin xyz=-0.4 -0.05 0.015 rpy=0 0 0
- joint bl_hip_joint: axis 0 -0.025319 0.99968 -> 0 0 -1; limit lower=-3.14 upper=3.14 effort=1000 velocity=20 -> lower=0 upper=${pi/2} effort=1000 velocity=100
- joint bl_knee_joint: limit lower=-3.14 upper=3.14 effort=1000 velocity=20 -> lower=0 upper=${pi} effort=1000 velocity=100
- joint bl_lat_joint: limit lower=-3.14 upper=3.14 effort=1000 velocity=20 -> lower=-0.5 upper=0.3 effort=1000 velocity=100
- joint br_hip_joint: axis 0 0 1 -> 0 0 -1; limit lower=-3.14 upper=3.14 effort=1000 velocity=20 -> lower=0 upper=${pi/2} effort=1000 velocity=100
- joint br_knee_joint: limit lower=-3.14 upper=3.14 effort=1000 velocity=20 -> lower=0 upper=${pi} effort=1000 velocity=100
- joint br_lat_joint: limit lower=-3.14 upper=3.14 effort=1000 velocity=20 -> lower=-0.5 upper=0.3 effort=1000 velocity=100
- joint fl_hip_joint: axis 0 0 1 -> 0 0 -1; limit lower=-3.14 upper=3.14 effort=1000 velocity=20 -> lower=0 upper=${pi/2} effort=1000 velocity=100
- joint fl_knee_joint: limit lower=-3.14 upper=3.14 effort=1000 velocity=20 -> lower=0 upper=${pi} effort=1000 velocity=100
- joint fl_lat_joint: limit lower=-3.14 upper=3.14 effort=1000 velocity=20 -> lower=-0.5 upper=0.3 effort=1000 velocity=100
- joint fr_hip_joint: axis 0 0 1 -> 0 0 -1; limit lower=-3.14 upper=3.14 effort=1000 velocity=20 -> lower=0 upper=${pi/2} effort=1000 velocity=100
- joint fr_knee_joint: limit lower=-3.14 upper=3.14 effort=1000 velocity=20 -> lower=0 upper=${pi} effort=1000 velocity=100
- joint fr_lat_joint: limit lower=-3.14 upper=3.14 effort=1000 velocity=20 -> lower=-0.5 upper=0.3 effort=1000 velocity=100
