Commit message: add ability to start simulation with laika flying

File: laika_ws/src/laika_sim/urdf/flying_laika.xacro.urdf (robot description, URDF)
Before this commit: robot laika, 14 links, 13 joints
Links:
- added link world
Joints:
- added joint world_to_base: type fixed, parent world, child base, origin xyz=0 0 1 rpy=0 0 0

Commit message: testing new pidf controller on fl joint

File: laika_ws/src/laika_sim/urdf/flying_laika.xacro.urdf (robot description, URDF)
Before this commit: robot laika, 15 links, 14 joints
Links:
- removed link bl_hip_link
- removed link bl_lower_link
- removed link bl_upper_link
- removed link br_hip_link
- removed link br_lower_link
- removed link br_upper_link
- removed link fr_hip_link
- removed link fr_lower_link
- removed link fr_upper_link
Joints:
- removed joint bl_hip_joint
- removed joint bl_knee_joint
- removed joint bl_lat_joint
- removed joint br_hip_joint
- removed joint br_knee_joint
- removed joint br_lat_joint
- removed joint fr_hip_joint
- removed joint fr_knee_joint
- removed joint fr_lat_joint
- joint fl_hip_joint: axis 0 0 1 -> 0 0 -1; limit lower=-3.14 upper=3.14 effort=1000 velocity=20 -> lower=0 upper=${pi/2} effort=1000 velocity=100
- joint fl_knee_joint: limit lower=-3.14 upper=3.14 effort=1000 velocity=20 -> lower=0 upper=${pi} effort=1000 velocity=100
- joint fl_lat_joint: limit lower=-3.14 upper=3.14 effort=1000 velocity=20 -> lower=-0.5 upper=0.3 effort=1000 velocity=100
- joint world_to_base: origin xyz=0 0 1 rpy=0 0 0 -> xyz=0 0 1 rpy=0 0 ${pi}

Commit message: pidf controll for all 4 joints (NOT TUNED)

File: laika_ws/src/laika_sim/urdf/flying_laika.xacro.urdf (robot description, URDF)
Before this commit: robot laika, 6 links, 5 joints
Links:
- added link bl_hip_link, mass 1.69584433341635; collision mesh filename=$(find laika_sim)/meshes/bl_hip_link.STL; visual mesh filename=$(find laika_sim)/meshes/bl_hip_link.STL
- added link bl_lower_link, mass 0.262408631372316; collision mesh filename=$(find laika_sim)/meshes/bl_lower_link.STL; visual mesh filename=$(find laika_sim)/meshes/bl_lower_link.STL
- added link bl_sphere; collision sphere radius=0.02; visual sphere radius=0.02
- added link bl_upper_link, mass 0.978822517757406; collision mesh filename=$(find laika_sim)/meshes/bl_upper_link.STL; visual mesh filename=$(find laika_sim)/meshes/bl_upper_link.STL
- added link br_hip_link, mass 1.69584433341635; collision mesh filename=$(find laika_sim)/meshes/br_hip_link.STL; visual mesh filename=$(find laika_sim)/meshes/br_hip_link.STL
- added link br_lower_link, mass 0.262408631372316; collision mesh filename=$(find laika_sim)/meshes/br_lower_link.STL; visual mesh filename=$(find laika_sim)/meshes/br_lower_link.STL
- added link br_sphere; collision sphere radius=0.02; visual sphere radius=0.02
- added link br_upper_link, mass 0.978822517757407; collision mesh filename=$(find laika_sim)/meshes/br_upper_link.STL; visual mesh filename=$(find laika_sim)/meshes/br_upper_link.STL
- added link fl_sphere; collision sphere radius=0.02; visual sphere radius=0.02
- added link fr_hip_link, mass 1.69584433341635; collision mesh filename=$(find laika_sim)/meshes/fr_hip_link.STL; visual mesh filename=$(find laika_sim)/meshes/fr_hip_link.STL
- added link fr_lower_link, mass 0.262408631372316; collision mesh filename=$(find laika_sim)/meshes/fr_lower_link.STL; visual mesh filename=$(find laika_sim)/meshes/fr_lower_link.STL
- added link fr_sphere; collision sphere radius=0.02; visual sphere radius=0.02
- added link fr_upper_link, mass 0.978822517757407; collision mesh filename=$(find laika_sim)/meshes/fl_upper_link.STL; visual mesh filename=$(find laika_sim)/meshes/fl_upper_link.STL
Joints:
- added joint bl_foot: type fixed, parent bl_lower_link, child bl_sphere, origin xyz=-0.4 -0.05 0.015 rpy=0 0 0
- added joint bl_hip_joint: type revolute, parent bl_hip_link, child bl_upper_link, origin xyz=0 -0.046 0.09 rpy=-0.025321 0 0, axis 0 0 -1, limit lower=0 upper=${pi/2} effort=1000 velocity=100
- added joint bl_knee_joint: type revolute, parent bl_upper_link, child bl_lower_link, origin xyz=0.35 -0.00013925 0.0054982 rpy=0.025295 -0.0011574 0.045716, axis 0 0 1, limit lower=0 upper=${pi} effort=1000 velocity=100
- added joint bl_lat_joint: type revolute, parent body_link, child bl_hip_link, origin xyz=0.043 0.3075 0.116 rpy=1.5708 0 1.5708, axis 1 0 0, limit lower=-0.5 upper=0.3 effort=1000 velocity=100
- added joint br_foot: type fixed, parent br_lower_link, child br_sphere, origin xyz=-0.4 -0.05 0.015 rpy=0 0 0
- added joint br_hip_joint: type revolute, parent br_hip_link, child br_upper_link, origin xyz=0 0.046 -0.126 rpy=0 0 3.1416, axis 0 0 -1, limit lower=0 upper=${pi/2} effort=1000 velocity=100
- added joint br_knee_joint: type revolute, parent br_upper_link, child br_lower_link, origin xyz=0.35 0 0.0055 rpy=0 0 0.04573, axis 0 0 1, limit lower=0 upper=${pi} effort=1000 velocity=100
- added joint br_lat_joint: type revolute, parent body_link, child br_hip_link, origin xyz=-0.043 0.3075 0.116 rpy=-1.5708 0 -1.5708, axis 1 0 0, limit lower=-0.5 upper=0.3 effort=1000 velocity=100
- added joint fl_foot: type fixed, parent fl_lower_link, child fl_sphere, origin xyz=-0.4 -0.05 0.015 rpy=0 0 0
- added joint fr_foot: type fixed, parent fr_lower_link, child fr_sphere, origin xyz=-0.4 -0.05 0.015 rpy=0 0 0
- added joint fr_hip_joint: type revolute, parent fr_hip_link, child fr_upper_link, origin xyz=0 0.046 -0.126 rpy=0 0 3.1416, axis 0 0 -1, limit lower=0 upper=${pi/2} effort=1000 velocity=100
- added joint fr_knee_joint: type revolute, parent fr_upper_link, child fr_lower_link, origin xyz=0.35 0 0.0055 rpy=0 0 0.04573, axis 0 0 1, limit lower=0 upper=${pi} effort=1000 velocity=100
- added joint fr_lat_joint: type revolute, parent body_link, child fr_hip_link, origin xyz=-0.043 -0.3075 0.116 rpy=-1.5708 0 -1.5708, axis 1 0 0, limit lower=-0.5 upper=0.3 effort=1000 velocity=100

Commit message: added slider config

File: laika_ws/src/laika_sim/urdf/flying_laika.xacro.urdf (robot description, URDF)
Before this commit: robot laika, 19 links, 18 joints
Joints:
- joint bl_hip_joint: limit lower=0 upper=${pi/2} effort=1000 velocity=100 -> lower=0 upper=${pi/2} effort=100 velocity=100
- joint bl_knee_joint: limit lower=0 upper=${pi} effort=1000 velocity=100 -> lower=0 upper=${pi} effort=100 velocity=100
- joint bl_lat_joint: limit lower=-0.5 upper=0.3 effort=1000 velocity=100 -> lower=-0.5 upper=0.3 effort=100 velocity=100
- joint br_hip_joint: limit lower=0 upper=${pi/2} effort=1000 velocity=100 -> lower=0 upper=${pi/2} effort=100 velocity=100
- joint br_knee_joint: limit lower=0 upper=${pi} effort=1000 velocity=100 -> lower=0 upper=${pi} effort=100 velocity=100
- joint br_lat_joint: limit lower=-0.5 upper=0.3 effort=1000 velocity=100 -> lower=-0.5 upper=0.3 effort=100 velocity=100
- joint fl_hip_joint: limit lower=0 upper=${pi/2} effort=1000 velocity=100 -> lower=0 upper=${pi/2} effort=100 velocity=100
- joint fl_knee_joint: limit lower=0 upper=${pi} effort=1000 velocity=100 -> lower=0 upper=${pi} effort=100 velocity=100
- joint fl_lat_joint: limit lower=-0.5 upper=0.3 effort=1000 velocity=100 -> lower=-0.5 upper=0.3 effort=100 velocity=100
- joint fr_hip_joint: limit lower=0 upper=${pi/2} effort=1000 velocity=100 -> lower=0 upper=${pi/2} effort=100 velocity=100
- joint fr_knee_joint: limit lower=0 upper=${pi} effort=1000 velocity=100 -> lower=0 upper=${pi} effort=100 velocity=100
- joint fr_lat_joint: limit lower=-0.5 upper=0.3 effort=1000 velocity=100 -> lower=-0.5 upper=0.3 effort=100 velocity=100

File: laika_ws/src/laika_sim/urdf/sliding_laika.xacro.urdf (robot description, URDF)
Before this commit: robot laika, 18 links, 17 joints
Links:
- removed link base
- added link slider, mass 100; visual box size=0.01 0.01 2.0
- added link world
Joints:
- removed joint base_to_body
- added joint slider_to_cart: type prismatic, parent slider, child body_link, origin xyz=0.0 0.0 0.0, axis 0 0 1, limit lower=-15 upper=15 effort=1000.0 velocity=30
- added joint world_to_base: type fixed, parent world, child slider, origin xyz=0 0 1 rpy=0 0 0
- joint bl_hip_joint: limit lower=0 upper=${pi/2} effort=100 velocity=100 -> lower=0 upper=${pi/2} effort=1000 velocity=100
- joint bl_knee_joint: limit lower=0 upper=${pi} effort=100 velocity=100 -> lower=0 upper=${pi} effort=1000 velocity=100
- joint bl_lat_joint: limit lower=-0.5 upper=0.3 effort=100 velocity=100 -> lower=-0.5 upper=0.3 effort=1000 velocity=100
- joint br_hip_joint: limit lower=0 upper=${pi/2} effort=100 velocity=100 -> lower=0 upper=${pi/2} effort=1000 velocity=100
- joint br_knee_joint: limit lower=0 upper=${pi} effort=100 velocity=100 -> lower=0 upper=${pi} effort=1000 velocity=100
- joint br_lat_joint: limit lower=-0.5 upper=0.3 effort=100 velocity=100 -> lower=-0.5 upper=0.3 effort=1000 velocity=100
- joint fl_hip_joint: limit lower=0 upper=${pi/2} effort=100 velocity=100 -> lower=0 upper=${pi/2} effort=1000 velocity=100
- joint fl_knee_joint: limit lower=0 upper=${pi} effort=100 velocity=100 -> lower=0 upper=${pi} effort=1000 velocity=100
- joint fl_lat_joint: limit lower=-0.5 upper=0.3 effort=100 velocity=100 -> lower=-0.5 upper=0.3 effort=1000 velocity=100
- joint fr_hip_joint: limit lower=0 upper=${pi/2} effort=100 velocity=100 -> lower=0 upper=${pi/2} effort=1000 velocity=100
- joint fr_knee_joint: limit lower=0 upper=${pi} effort=100 velocity=100 -> lower=0 upper=${pi} effort=1000 velocity=100
- joint fr_lat_joint: limit lower=-0.5 upper=0.3 effort=100 velocity=100 -> lower=-0.5 upper=0.3 effort=1000 velocity=100
