Commit message: new branch for testing on knee only

File: laika_ws/src/laika_sim/urdf/sliding_laika.xacro.urdf (robot description, URDF)
Before this commit: robot laika, 19 links, 18 joints
Joints:
- joint bl_hip_joint: axis 0 0 -1 -> (none); limit lower=0 upper=${pi/2} effort=1000 velocity=100 -> (none); type revolute -> fixed
- joint bl_lat_joint: axis 1 0 0 -> (none); limit lower=-0.5 upper=0.3 effort=1000 velocity=100 -> (none); type revolute -> fixed
- joint br_hip_joint: axis 0 0 -1 -> (none); limit lower=0 upper=${pi/2} effort=1000 velocity=100 -> (none); type revolute -> fixed
- joint br_lat_joint: axis 1 0 0 -> (none); limit lower=-0.5 upper=0.3 effort=1000 velocity=100 -> (none); type revolute -> fixed
- joint fl_hip_joint: axis 0 0 -1 -> (none); limit lower=0 upper=${pi/2} effort=1000 velocity=100 -> (none); type revolute -> fixed
- joint fl_lat_joint: axis 1 0 0 -> (none); limit lower=-0.5 upper=0.3 effort=1000 velocity=100 -> (none); type revolute -> fixed
- joint fr_hip_joint: axis 0 0 -1 -> (none); limit lower=0 upper=${pi/2} effort=1000 velocity=100 -> (none); type revolute -> fixed
- joint fr_lat_joint: axis 1 0 0 -> (none); limit lower=-0.5 upper=0.3 effort=1000 velocity=100 -> (none); type revolute -> fixed
