Commit message: ik node created

File: laika_ws/src/laika_sim/urdf/test_stand_laika_left.xacro.urdf (robot description, URDF)
Before this commit: robot laika, 6 links, 5 joints
Links:
- removed link fr_hip_link
- removed link fr_lower_link
- removed link fr_sphere
- removed link fr_upper_link
- added link fl_hip_link, mass 1.6958; collision mesh filename=$(find laika_sim)/meshes/fl_hip_link.STL; visual mesh filename=$(find laika_sim)/meshes/fl_hip_link.STL
- added link fl_lower_link, mass 0.262408631372316; collision mesh filename=$(find laika_sim)/meshes/fl_lower_link.STL; visual mesh filename=$(find laika_sim)/meshes/fl_lower_link.STL
- added link fl_sphere; collision sphere radius=0.02; visual sphere radius=0.02
- added link fl_upper_link, mass 0.97882; collision mesh filename=$(find laika_sim)/meshes/fl_upper_link.STL; visual mesh filename=$(find laika_sim)/meshes/fl_upper_link.STL
Joints:
- removed joint fr_foot
- removed joint fr_hip_joint
- removed joint fr_knee_joint
- added joint fl_foot: type fixed, parent fl_lower_link, child fl_sphere, origin xyz=-0.4 -0.05 0.015 rpy=0 0 0
- added joint fl_hip_joint: type revolute, parent fl_hip_link, child fl_upper_link, origin xyz=0 -0.046 0.09 rpy=0 0 0, axis 0 0 -1, limit lower=0 upper=${pi/2} effort=1000 velocity=100
- added joint fl_knee_joint: type revolute, parent fl_upper_link, child fl_lower_link, origin xyz=0.35 0 0.0055 rpy=0 0 0.04573, axis 0 0 1, limit lower=0 upper=${pi} effort=1000 velocity=100
- joint slider_to_cart: child fr_hip_link -> fl_hip_link; origin xyz=0.0 0.0 0.0 rpy=0 0 0 -> xyz=0.0 0.0 0.0 rpy=1.5708 0 0
