Commit message: dummy ik path added

File: laika_ws/src/laika_sim/urdf/test_stand_laika.xacro.urdf (robot description, URDF)
Before this commit: robot laika, 6 links, 5 joints
Joints:
- joint fr_hip_joint: limit lower=0 upper=${2*pi} effort=1000 velocity=100 -> lower=${-pi} upper=${2*pi} effort=1000 velocity=100
- joint fr_knee_joint: origin xyz=0.35 0 0.0055 rpy=0 0 0.04573 -> xyz=0.35 0 0.0055 rpy=0 0 0
- joint slider_to_cart: origin xyz=0.0 0.0 0.0 rpy=0 0 0 -> xyz=0.0 0.0 0.0 rpy=-1.5708 0 0

Commit message: MPC jumping implemented

File: laika_ws/src/laika_sim/urdf/test_stand_laika.xacro.urdf (robot description, URDF)
Before this commit: robot laika, 6 links, 5 joints
Links:
- link fr_upper_link: geometry collision mesh filename=$(find laika_sim)/meshes/fr_upper_link.STL; visual mesh filename=$(find laika_sim)/meshes/fr_upper_link.STL

Commit message: urdffing

File: laika_ws/src/laika_sim/urdf/test_stand_laika.xacro.urdf (robot description, URDF)
Before this commit: robot laika, 6 links, 5 joints
Links:
- link fr_hip_link: mass 1.69584433341635 -> 2.69584433341635
Joints:
- joint fr_hip_joint: limit lower=${-pi} upper=${2*pi} effort=1000 velocity=100 -> lower=${-pi} upper=${2*pi} effort=120 velocity=20
- joint fr_knee_joint: limit lower=0 upper=${2*pi} effort=1000 velocity=100 -> lower=0 upper=${2*pi} effort=120 velocity=20
