Commit message: cleaned up xacro files

File: laika_ws/src/laika_description/xacro/leg.xacro (robot description, xacro)
@@ -2,13 +2,13 @@
 <robot xmlns:xacro="http://www.ros.org/wiki/xacro">
   <!-- Left Leg Macro -->
-  <xacro:macro name="left_leg" params="name *origin">
+  <xacro:macro name="leg" params="*origin">
     <!-- base link -->
-    <joint name="base_to_${name}_hip" type="fixed">
+    <joint name="base_to_hip" type="fixed">
       <xacro:insert_block name="origin"/>
       <parent link="base"/>
-      <child link="${name}_hip_link"/>
+      <child link="hip_link"/>
     </joint>
     <!-- Hip Link -->
-    <link name="${name}_hip_link">
+    <link name="hip_link">
       <visual>
         <origin xyz="-2.18152e-18 5.38878e-34 -8.80055e-18" rpy="6.12323e-17 -0 0"/>
@@ -31,5 +31,5 @@
     </link>
     <!-- Upper Leg Link -->
-    <link name="${name}_upper_leg_link">
+    <link name="upper_leg_link">
       <visual>
         <origin xyz="6.50521e-18 1.38778e-17 -0.0175" rpy="1.5708 -6.82067e-39 0"/>
@@ -52,5 +52,5 @@
     </link>
     <!-- Lower Leg Link -->
-    <link name="${name}_lower_leg_link">
+    <link name="lower_leg_link">
       <visual>
         <origin xyz="0 -0.07 -0.0105" rpy="-1.5708 -1.10793e-33 0"/>
@@ -73,8 +73,8 @@
     </link>
     <!-- Hip Joint -->
-    <joint name="${name}_hip_joint" type="revolute">
+    <joint name="hip_joint" type="revolute">
       <origin xyz="-7.11766e-17 -0.106 -0.0495" rpy="-1.5708 1.01231e-16 -2.87032e-22"/>
-      <parent link="${name}_hip_link"/>
-      <child link="${name}_upper_leg_link"/>
+      <parent link="hip_link"/>
+      <child link="upper_leg_link"/>
       <axis xyz="0 0 1"/>
       <limit effort="1000" lower="0" upper="${pi/2}" velocity="10"/>
@@ -82,8 +82,8 @@
     </joint>
     <!-- Knee Joint -->
-    <joint name="${name}_knee_joint" type="revolute">
+    <joint name="knee_joint" type="revolute">
       <origin xyz="0.35 1.59595e-16 -0.028" rpy="-3.14159 1.11613e-17 1.67306e-17"/>
-      <parent link="${name}_upper_leg_link"/>
-      <child link="${name}_lower_leg_link"/>
+      <parent link="upper_leg_link"/>
+      <child link="lower_leg_link"/>
       <axis xyz="0 0 1"/>
       <limit effort="1000" lower="0" upper="${pi}" velocity="10"/>

File: laika_ws/src/laika_description/xacro/robot.xacro (robot description, xacro)
@@ -7,5 +7,5 @@
     <xacro:include filename="$(find laika_description)/xacro/const.xacro"/>
     <xacro:include filename="$(find laika_description)/xacro/materials.xacro"/>
-    <xacro:include filename="$(find laika_description)/xacro/left_leg.xacro"/>
+    <xacro:include filename="$(find laika_description)/xacro/leg.xacro"/>
     <!-- fly -->
     <xacro:if value="$(arg fly)">
@@ -49,34 +49,18 @@
     <!-- legs -->
     <xacro:if value="$(arg leg_only)">
-      <xacro:left_leg name="left">
+      <xacro:leg>
         <origin xyz="0 0 0" rpy="0 0 ${-pi/2}"/>
-      </xacro:left_leg>
+      </xacro:leg>
     </xacro:if>
-    <!-- simulation -->
-    <xacro:if value="$(arg simulation)">
-      <xacro:if value="$(arg leg_only)">
-        <ros2_control name="GazeboSystem" type="system">
-          <hardware>
-            <plugin>gz_ros2_control/GazeboSimSystem</plugin>
-          </hardware>
-          <joint name="left_hip_joint">
-            <command_interface name="effort" />
-            <state_interface name="position" />
-            <state_interface name="velocity" />
-            <state_interface name="effort" />
-          </joint>
-          <joint name="left_knee_joint">
-            <command_interface name="effort" />
-            <state_interface name="position" />
-            <state_interface name="velocity" />
-            <state_interface name="effort" />
-          </joint>
-        </ros2_control>
+    <!-- leg only -->
+    <xacro:if value="$(arg leg_only)">
+      <!-- simulation -->
+      <xacro:if value="$(arg simulation)">
+        <xacro:include filename="$(find laika_description)/xacro/leg_gazebo.xacro"/>
       </xacro:if>
-      <gazebo>
-        <plugin filename="libgz_ros2_control-system.so" name="gz_ros2_control::GazeboSimROS2ControlPlugin">
-          <parameters>$(find laika_sim)/config/laika_controller.yaml</parameters>
-        </plugin>
-      </gazebo>
-  </xacro:if>
+      <!-- real -->
+      <xacro:unless value="$(arg simulation)">
+        <xacro:include filename="$(find laika_description)/xacro/leg_ros2_control.xacro"/>
+      </xacro:unless>
+    </xacro:if>
 </robot>
