Commit message: use current leg design in simulation

File: laika_ws/src/laika_description/xacro/robot.xacro (robot description, xacro)
@@ -7,5 +7,5 @@
     <xacro:include filename="$(find laika_description)/xacro/const.xacro"/>
     <xacro:include filename="$(find laika_description)/xacro/materials.xacro"/>
-    <xacro:include filename="$(find laika_description)/xacro/leg.xacro"/>
+    <xacro:include filename="$(find laika_description)/xacro/leg_current.xacro"/>
     <!-- fly -->
     <xacro:if value="$(arg fly)">
@@ -50,5 +50,6 @@
     <xacro:if value="$(arg leg_only)">
       <xacro:leg>
-        <origin xyz="0 0 0" rpy="0 0 ${-pi/2}"/>
+        <!-- <origin xyz="0 0 0" rpy="0 0 ${-pi/2}"/> -->
+        <origin xyz="0 0 0" rpy="${pi/2} 0 ${-pi/2}"/>
       </xacro:leg>
     </xacro:if>
