Commit message: ik working irl

File: laika_ws/src/laika_description/xacro/leg_current.xacro (robot description, xacro)
@@ -75,5 +75,5 @@
       <child link="upper_link"/>
       <axis xyz="0 0 -1"/>
-      <limit effort="1000" lower="0" upper="${pi/2}" velocity="100"/>
+      <limit effort="1000" lower="${-pi/4}" upper="${pi/2}" velocity="100"/>
       <dynamics damping="${hip_damping}" friction="${hip_friction}"/>
     </joint>

File: laika_ws/src/laika_description/xacro/leg_ros2_control.xacro (robot description, xacro)
@@ -8,5 +8,5 @@
     <joint name="hip_joint">
       <param name="can_id">1</param>
-      <param name="motor_current_limit">5</param>
+      <param name="motor_current_limit">0</param>
       <command_interface name="effort" data_type="double"/>
       <state_interface name="position" data_type="double"/>
@@ -16,5 +16,5 @@
     <joint name="knee_joint">
       <param name="can_id">2</param>
-      <param name="motor_current_limit">5</param>
+      <param name="motor_current_limit">0</param>
       <command_interface name="effort" data_type="double"/>
       <state_interface name="position" data_type="double"/>
