Commit message: feat: added rl control

File: laika_ws/src/laika_description/xacro/leg_current.xacro (robot description, xacro)
@@ -86,4 +86,19 @@
       <dynamics damping="${knee_damping}" friction="${knee_friction}"/>
     </joint>
+    <!-- This is a dummy link for software to know where the tip of the leg is -->
+    <!-- Tiny mass so that physics doesn't break -->
+    <!-- <link name="foot_link"> -->
+    <!--   <inertial> -->
+    <!--     <mass value="0.001"/> -->
+    <!--     <inertia ixx="1e-6" ixy="0" ixz="0" iyy="1e-6" iyz="0" izz="1e-6"/> -->
+    <!--   </inertial> -->
+    <!-- </link> -->
+    <!---->
+    <!-- <joint name="lower_to_foot" type="fixed"> -->
+    <!--   <parent link="lower_link"/> -->
+    <!--   <child link="foot_link"/> -->
+    <!--   <origin xyz="-0.4 -0.05 0" rpy="0 0 0"/>  -->
+    <!-- </joint> -->
+    <!---->
   </xacro:macro>
 </robot>
