Commit message: added force correction at foot

File: laika_ws/src/laika_description/xacro/const.xacro (robot description, xacro)
@@ -6,7 +6,7 @@
   <xacro:property name="lower_leg_mass" value="1.0" />
   <!-- damping and friction -->
-  <xacro:property name="hip_damping" value="0.2" />
+  <xacro:property name="hip_damping" value="0.01" />
   <xacro:property name="hip_friction" value="0.01" />
-  <xacro:property name="knee_damping" value="0.2" />
+  <xacro:property name="knee_damping" value="0.01" />
   <xacro:property name="knee_friction" value="0.01" />
 </robot>
